Commit message: cloned udacity_bot to rob_bot, ready to edit

File: src/rob_bot/urdf/rob_bot.xacro (robot description, xacro)
@@ -1,6 +1,6 @@
 <?xml version='1.0'?>
-<robot name="udacity_bot"
+<robot name="rob_bot"
     xmlns:xacro="http://www.ros.org/wiki/xacro">
-    <xacro:include filename="$(find udacity_bot)/urdf/udacity_bot.gazebo" />
+    <xacro:include filename="$(find rob_bot)/urdf/rob_bot.gazebo" />
     <link name="robot_footprint"></link>
     <joint name="robot_footprint_joint" type="fixed">
@@ -163,5 +163,5 @@
             <origin xyz="0 0 0" rpy="0 0 0"/>
             <geometry>
-                <mesh filename="package://udacity_bot/meshes/hokuyo.dae"/>
+                <mesh filename="package://rob_bot/meshes/hokuyo.dae"/>
             </geometry>
         </visual>

Commit message: completed second model

File: src/rob_bot/urdf/rob_bot.xacro (robot description, xacro)
@@ -9,4 +9,5 @@
         <child link="chassis" />
     </joint>
+    <!-- Chassis -->
     <link name='chassis'>
         <pose>0 0 0.1 0 0 0</pose>
@@ -16,5 +17,5 @@
             <inertia ixx="0.1" ixy="0" ixz="0" iyy="0.1" iyz="0" izz="0.1" />
         </inertial>
-        <collision name='collision'>
+        <collision name='chassis_collision'>
             <origin xyz="0 0 0" rpy=" 0 0 0"/>
             <geometry>
@@ -28,83 +29,126 @@
             </geometry>
         </visual>
-        <collision name='back_caster_collision'>
-            <origin xyz="-0.15 0 -0.05" rpy=" 0 0 0"/>
-            <geometry>
-                <sphere radius="0.0499"/>
-            </geometry>
-        </collision>
-        <visual name='back_caster_visual'>
-            <origin xyz="-0.15 0 -0.05" rpy=" 0 0 0"/>
-            <geometry>
-                <sphere radius="0.05"/>
-            </geometry>
-        </visual>
-        <collision name='front_caster_collision'>
-            <origin xyz="0.15 0 -0.05" rpy=" 0 0 0"/>
-            <geometry>
-                <sphere radius="0.0499"/>
-            </geometry>
-        </collision>
-        <visual name='front_caster_visual'>
-            <origin xyz="0.15 0 -0.05" rpy=" 0 0 0"/>
-            <geometry>
-                <sphere radius="0.05"/>
-            </geometry>
-        </visual>
-    </link>
-    <link name='left_wheel'>
-        <visual name='left_wheel_visual'>
-            <origin xyz="0 0 0" rpy="0 1.5707 1.5707"/>
-            <geometry>
-                <cylinder radius="0.1" length='0.05'/>
-            </geometry>
-        </visual>
-        <inertial>
-            <mass value="5.0"/>
-            <origin xyz="0.0 0 0" rpy="0 1.5707 1.5707"/>
-            <inertia ixx="0.1" ixy="0" ixz="0" iyy="0.1" iyz="0" izz="0.1"/>
-        </inertial>
-        <collision name='collision'>
-            <origin xyz="0 0 0" rpy="0 1.5707 1.5707"/>
-            <geometry>
-                <cylinder radius="0.1" length='0.05'/>
-            </geometry>
-        </collision>
-    </link>
-    <link name='right_wheel'>
-        <visual name='left_wheel_visual'>
-            <origin xyz="0 0 0" rpy="0 1.5707 1.5707"/>
-            <geometry>
-                <cylinder radius="0.1" length='0.05'/>
-            </geometry>
-        </visual>
-        <inertial>
-            <mass value="5.0"/>
-            <origin xyz="0.0 0 0" rpy="0 1.5707 1.5707"/>
-            <inertia ixx="0.1" ixy="0" ixz="0" iyy="0.1" iyz="0" izz="0.1"/>
-        </inertial>
-        <collision name='collision'>
-            <origin xyz="0 0 0" rpy="0 1.5707 1.5707"/>
-            <geometry>
-                <cylinder radius="0.1" length='0.05'/>
-            </geometry>
-        </collision>
-    </link>
-    <joint type="continuous" name="left_wheel_hinge">
-        <origin xyz="0 0.15 0" rpy="0 0 0"/>
-        <child link="left_wheel"/>
-        <parent link="chassis"/>
-        <axis xyz="0 1 0" rpy="0 0 0"/>
-        <limit effort="10000" velocity="1000"/>
-        <dynamics damping="1.0" friction="1.0"/>
-    </joint>
-    <joint type="continuous" name="right_wheel_hinge">
-        <origin xyz="0 -0.15 0" rpy="0 0 0"/>
-        <child link="right_wheel"/>
-        <parent link="chassis"/>
-        <axis xyz="0 1 0" rpy="0 0 0"/>
-        <limit effort="10000" velocity="1000"/>
-        <dynamics damping="1.0" friction="1.0"/>
-    </joint>
+    </link>
+    <!-- end chassis -->
+    <!-- front left wheel -->
+    <link name="front_left_wheel">
+        <visual name='front_left_wheel_visual'>
+            <origin xyz="0 0 0" rpy=" 0 1.5707 1.5707"/>
+            <geometry>
+                <cylinder radius="0.1" length="0.05"/>
+            </geometry>
+            <material name="black"/>
+        </visual>
+        <collision name='front_left_wheel_collision'>
+            <origin xyz="0 0 0" rpy=" 0 1.5707 1.5707"/>
+            <geometry>
+                <cylinder radius="0.1" length="0.05"/>
+            </geometry>
+        </collision>
+        <inertial>
+            <mass value="5.0"/>
+            <origin xyz="0.0 0 0" rpy=" 0 1.5707 1.5707"/>
+            <inertia ixx="0.1" ixy="0" ixz="0" iyy="0.1" iyz="0" izz="0.1" />
+        </inertial>
+    </link>
+    <joint type="continuous" name="front_left_wheel_joint">
+        <origin xyz="0.15 0.18 -.05" rpy="0 0 0"/>
+        <child link="front_left_wheel"/>
+        <parent link="chassis"/>
+        <axis xyz="0 1 0" rpy="0 0 0"/>
+        <limit effort="10000" velocity="1000"/>
+        <joint_properties damping="1.0" friction="1.0"/>
+    </joint>
+    <!-- end front left wheel -->
+    <!-- front right wheel -->
+    <link name="front_right_wheel">
+        <visual name='front_right_wheel_visual'>
+            <origin xyz="0 0 0" rpy=" 0 1.5707 1.5707"/>
+            <geometry>
+                <cylinder radius="0.1" length="0.05"/>
+            </geometry>
+            <material name="black"/>
+        </visual>
+        <collision name='front_right_wheel_collision'>
+            <origin xyz="0 0 0" rpy=" 0 1.5707 1.5707"/>
+            <geometry>
+                <cylinder radius="0.1" length="0.05"/>
+            </geometry>
+        </collision>
+        <inertial>
+            <mass value="5.0"/>
+            <origin xyz="0.0 0 0" rpy=" 0 1.5707 1.5707"/>
+            <inertia ixx="0.1" ixy="0" ixz="0" iyy="0.1" iyz="0" izz="0.1" />
+        </inertial>
+    </link>
+    <joint type="continuous" name="front_right_wheel_joint">
+        <origin xyz="-0.15 0.18 -.05" rpy="0 0 0"/>
+        <child link="front_right_wheel"/>
+        <parent link="chassis"/>
+        <axis xyz="0 1 0" rpy="0 0 0"/>
+        <limit effort="10000" velocity="1000"/>
+        <joint_properties damping="1.0" friction="1.0"/>
+    </joint>
+    <!-- end front right wheel -->
+    <!-- rear left wheel -->
+    <link name="rear_left_wheel">
+        <visual name='rear_left_wheel_visual'>
+            <origin xyz="0 0 0" rpy=" 0 1.5707 1.5707"/>
+            <geometry>
+                <cylinder radius="0.1" length="0.05"/>
+            </geometry>
+            <material name="black"/>
+        </visual>
+        <collision name='rear_left_wheel_collision'>
+            <origin xyz="0 0 0" rpy=" 0 1.5707 1.5707"/>
+            <geometry>
+                <cylinder radius="0.1" length="0.05"/>
+            </geometry>
+        </collision>
+        <inertial>
+            <mass value="5.0"/>
+            <origin xyz="0.0 0 0" rpy=" 0 1.5707 1.5707"/>
+            <inertia ixx="0.1" ixy="0" ixz="0" iyy="0.1" iyz="0" izz="0.1" />
+        </inertial>
+    </link>
+    <joint type="continuous" name="rear_left_wheel_joint">
+        <origin xyz="0.15 -0.18 -0.05" rpy="0 0 0"/>
+        <child link="rear_left_wheel"/>
+        <parent link="chassis"/>
+        <axis xyz="0 1 0" rpy="0 0 0"/>
+        <limit effort="10000" velocity="1000"/>
+        <joint_properties damping="1.0" friction="1.0"/>
+    </joint>
+    <!-- end rear left wheel -->
+    <!-- rear right wheel -->
+    <link name="rear_right_wheel">
+        <visual name='rear_right_wheel_visual'>
+            <origin xyz="0 0 0" rpy=" 0 1.5707 1.5707"/>
+            <geometry>
+                <cylinder radius="0.1" length="0.05"/>
+            </geometry>
+            <material name="black"/>
+        </visual>
+        <collision name='rear_right_wheel_collision'>
+            <origin xyz="0 0 0" rpy=" 0 1.5707 1.5707"/>
+            <geometry>
+                <cylinder radius="0.1" length="0.05"/>
+            </geometry>
+        </collision>
+        <inertial>
+            <mass value="5.0"/>
+            <origin xyz="0.0 0 0" rpy=" 0 1.5707 1.5707"/>
+            <inertia ixx="0.1" ixy="0" ixz="0" iyy="0.1" iyz="0" izz="0.1" />
+        </inertial>
+    </link>
+    <joint type="continuous" name="rear_right_wheel_joint">
+        <origin xyz="-0.15 -0.18 -0.05" rpy="0 0 0"/>
+        <child link="rear_right_wheel"/>
+        <parent link="chassis"/>
+        <axis xyz="0 1 0" rpy="0 0 0"/>
+        <limit effort="10000" velocity="1000"/>
+        <joint_properties damping="1.0" friction="1.0"/>
+    </joint>
+    <!-- end rear right wheel -->
     <link name='camera'>
         <visual name='camera_visual'>
@@ -131,11 +175,9 @@
         <parent link="chassis"/>
     </joint>
-<!-- begin customisation -->
-<!--
-        <link name='rear_fin'>
-        <visual name='rear_fin'>
-            <origin xyz="0 0 0" rpy="0 0 0"/>
-            <geometry>
-                <box size='0.05 .2 0.3'/>
+    <link name='hokuyo'>
+        <visual name='hokuyo_visual'>
+            <origin xyz="0 0 0" rpy="0 0 0"/>
+            <geometry>
+                <mesh filename="package://rob_bot/meshes/hokuyo.dae"/>
             </geometry>
         </visual>
@@ -148,30 +190,4 @@
             <origin xyz="0 0 0" rpy="0 0 0"/>
             <geometry>
-                <box size='0.05 .2 0.3'/>
-            </geometry>
-        </collision>
-    </link>
-    <joint type="fixed" name="rear_fin_joint">
-        <origin xyz="-0.2 0 0.05" rpy="0 0 0"/>
-        <child link="rear_fin"/>
-        <parent link="chassis"/>
-    </joint>
-    -->
-<!-- end customisation -->
-    <link name='hokuyo'>
-        <visual name='hokuyo_visual'>
-            <origin xyz="0 0 0" rpy="0 0 0"/>
-            <geometry>
-                <mesh filename="package://rob_bot/meshes/hokuyo.dae"/>
-            </geometry>
-        </visual>
-        <inertial>
-            <mass value="0.1"/>
-            <origin xyz="0.0 0 0" rpy="0 0 0"/>
-            <inertia ixx="1e-6" ixy="0" ixz="0" iyy="1e-6" iyz="0" izz="1e-6"/>
-        </inertial>
-        <collision name='collision'>
-            <origin xyz="0 0 0" rpy="0 0 0"/>
-            <geometry>
                 <box size='0.1 0.1 0.1'/>
             </geometry>
